File: CHV_DC31.kicad_pcb (KiCad board)
At the start: 2 copper layers, 98.1 x 91.7 mm, 84 parts, among them IC1 W25Q16JVUXIQ_TR, J1 USB_C_Receptacle_USB2.0, J2 Conn_01x02, J3 Conn_02x03_Odd_Even, J4 Conn_02x03_Odd_Even, J5 Conn_02x03_Odd_Even, J6 Conn_01x03, SW2 SW_SPST, SW3 SW_SPST, SW4 SW_SPST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

Commit message: updates
Parts:
- J2: footprint Connector_PinHeader_2.54mm:PinHeader_1x02_P2.54mm_Vertical -> Jumper:SolderJumper-2_P1.3mm_Open_Pad1.0x1.5mm
- moved J6 104.3 mm to (133.5, 134.5), turned to -90 degrees
- moved SW6 80.1 mm to (89.1, 76.5)
- moved R6 77.5 mm to (139.8, 118.2), turned to 45 degrees
- moved R5 75.7 mm to (141.2, 119.6), turned to 45 degrees
- moved C1 67.1 mm to (141.5, 113.1), turned to 45 degrees
- moved IC1 66.8 mm to (139.2, 109.0), turned to -90 degrees
- moved C17 62.3 mm to (147.9, 98.3), turned to 45 degrees
- moved J2 60.1 mm to (158.2, 107.6), turned to -90 degrees
- moved C3 58.2 mm to (155.9, 104.8), turned to -135 degrees
- moved R2 53.3 mm to (155.8, 110.6), turned to 45 degrees
- moved C18 51.5 mm to (152.1, 98.4), turned to -45 degrees
- moved C8 49.2 mm to (152.6, 114.3), turned to -45 degrees
- moved C11 43.5 mm to (154.4, 103.4), turned to 45 degrees
- moved C15 43.4 mm to (151.1, 115.8), turned to -45 degrees
- moved C9 43.2 mm to (154.1, 112.9)
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Connections:
- U3 pad 12: unconnected-(U3-Pad12) -> RP1_LED_3
- U3 pad 15: unconnected-(U3-Pad15) -> RP1_LED_1
- U3 pad 16: unconnected-(U3-Pad16) -> RP1_LED_2
- U3 pad 27: RP1_CAN_TX -> unconnected-(U3-GPIO16-Pad27)
- U3 pad 28: RP1_CAN_RX -> unconnected-(U3-GPIO17-Pad28)
- U3 pad 5: unconnected-(U3-Pad5) -> RP1_CAN_RX
- U3 pad 6: unconnected-(U3-Pad6) -> RP1_CAN_TX
- U3 pad 7: RP1_LED_1 -> unconnected-(U3-GPIO5-Pad7)
- U3 pad 8: RP1_LED_2 -> unconnected-(U3-GPIO6-Pad8)
- U3 pad 9: RP1_LED_3 -> unconnected-(U3-GPIO7-Pad9)
Routing:
- net +3V3: track 0.00 -> 29.8 mm
- net RP1_v1: track 0.00 -> 11.2 mm
- net GND: track 0.00 -> 10.8 mm
- net RP1_XTAL_OUT: track 0.00 -> 9.73 mm
- net RP1_XTAL_IN: track 0.00 -> 9.29 mm
- net RP1_USB_D-: track 0.00 -> 8.93 mm
- net RP1_USB_D+: track 0.00 -> 8.92 mm
- net RP1_QSPI_CS: track 0.00 -> 8.51 mm
- net RP1_QSPI_SD3: track 0.00 -> 8.35 mm
- net RP1_QSPI_SD1: track 0.00 -> 8.27 mm
- net RP1_QSPI_SD2: track 0.00 -> 7.75 mm
- net RP1_QSPI_SD0: track 0.00 -> 7.46 mm
- net RP1_QSPI_SCLK: track 0.00 -> 7.26 mm
- net RP1_SWD: track 0.00 -> 7.18 mm
- net RP1_SWCLK: track 0.00 -> 7.05 mm
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- added copper zone on B.Cu, net GND

Commit message: layed out led ring
Parts:
- removed D4, D5, D6, D7, D8: LED, LED_SMD:LED_1206_3216Metric
- removed R12, R13, R14, R15, R16: R, Resistor_SMD:R_0805_2012Metric
- added D15: LED, LED_SMD:LED_1206_3216Metric, B.Cu at (122.0, 102.6)
- added D16: LED, LED_SMD:LED_1206_3216Metric, B.Cu at (124.3, 115.5)
- added D17: LED, LED_SMD:LED_1206_3216Metric, B.Cu at (134.3, 107.1)
- added D18: LED, LED_SMD:LED_1206_3216Metric, B.Cu at (126.8, 100.9)
- added D19: LED, LED_SMD:LED_1206_3216Metric, B.Cu at (120.3, 112.2)
- added D20: LED, LED_SMD:LED_1206_3216Metric, B.Cu at (133.4, 112.2)
- added D21: LED, LED_SMD:LED_1206_3216Metric, B.Cu at (131.8, 102.6)
- added D22: LED, LED_SMD:LED_1206_3216Metric, B.Cu at (119.4, 107.0)
- added D23: LED, LED_SMD:LED_1206_3216Metric, B.Cu at (129.4, 115.5)
- added R24: R, Resistor_SMD:R_0805_2012Metric, B.Cu at (118.8, 99.2)
- added R25: R, Resistor_SMD:R_0805_2012Metric, B.Cu at (125.0, 106.8)
- added R26: R, Resistor_SMD:R_0805_2012Metric, B.Cu at (125.5, 111.8)
- added R27: R, Resistor_SMD:R_0805_2012Metric, B.Cu at (122.9, 98.9)
- added R28: R, Resistor_SMD:R_0805_2012Metric, B.Cu at (116.8, 109.9)
- added R29: R, Resistor_SMD:R_0805_2012Metric, B.Cu at (128.0, 109.7)
- added R30: R, Resistor_SMD:R_0805_2012Metric, B.Cu at (135.6, 101.3)
- added R31: R, Resistor_SMD:R_0805_2012Metric, B.Cu at (122.3, 108.8)
- added R32: R, Resistor_SMD:R_0805_2012Metric, B.Cu at (126.9, 119.0)
- moved R23 27.7 mm to (208.2, 123.0)
- moved U1 5.60 mm to (143.3, 98.1)
- moved C12 0.49 mm to (145.2, 103.4)
Connections:
- U3 pad 12: RP1_LED_3 -> unconnected-(U3-GPIO9-Pad12)
- U3 pad 13: RP1_LED_4 -> unconnected-(U3-GPIO10-Pad13)
- U3 pad 14: RP1_LED_5 -> RP1_CAN_RX
- U3 pad 15: RP1_LED_1 -> RP1_CAN_TX
- U3 pad 16: RP1_LED_2 -> unconnected-(U3-GPIO13-Pad16)
- U3 pad 5: RP1_CAN_RX -> LED_LINE_4
- U3 pad 6: RP1_CAN_TX -> LED_LINE_3
- U3 pad 7: unconnected-(U3-GPIO5-Pad7) -> LED_LINE_2
- U3 pad 8: unconnected-(U3-GPIO6-Pad8) -> LED_LINE_1
Routing:
- net LED_LINE_2: track 0.00 -> 54.1 mm
- net LED_LINE_1: track 0.00 -> 47.9 mm
- net LED_LINE_3: track 0.00 -> 43.1 mm
- net LED_LINE_4: track 0.00 -> 35.6 mm
- net Net-(D17-A): track 0.00 -> 24.3 mm
- net Net-(J1-D--PadA7): track 0.00 -> 21.8 mm
- net Net-(J1-D+-PadA6): track 0.00 -> 21.3 mm
- net Net-(D16-A): track 0.00 -> 20.4 mm
- net Net-(D20-A): track 0.00 -> 6.95 mm
- net RP1_CAN_RX: track 6.03 -> 0.00 mm
- net Net-(D19-A): track 0.00 -> 3.68 mm
- net Net-(D23-A): track 0.00 -> 3.67 mm
- net Net-(D15-A): track 0.00 -> 3.60 mm
- net Net-(D22-A): track 0.00 -> 3.38 mm
- net Net-(D18-A): track 0.00 -> 2.92 mm
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
Commit message: power
Parts:
- moved D1 94.6 mm to (135.6, 130.0)
- moved R23 91.9 mm to (116.3, 122.5), turned to 135 degrees
- moved R4 85.2 mm to (129.7, 125.2), turned to 45 degrees
- moved C2 82.1 mm to (145.3, 126.8), turned to 45 degrees
- moved U2 77.2 mm to (143.3, 124.5), turned to 45 degrees
- moved R9 75.2 mm to (140.5, 127.2), turned to 135 degrees
- moved C10 73.5 mm to (145.9, 121.8), turned to 135 degrees
- moved R1 51.3 mm to (147.7, 92.7), turned to 45 degrees
- moved R3 47.9 mm to (131.8, 127.1), turned to 45 degrees
- moved SW7 18.0 mm to (113.8, 126.6), turned to 135 degrees
Routing:
- net VBUS: track 0.00 -> 50.1 mm
- net Net-(J6-Pin_3): track 0.00 -> 30.2 mm
- net Net-(J6-Pin_2): track 0.00 -> 28.3 mm
- net +3V3: track 30.0 -> 54.0 mm
- net Net-(D1-A): track 0.00 -> 17.6 mm
- net RP1_CAN_TX: track 0.00 -> 7.88 mm
- net Net-(J1-CC2): track 0.00 -> 7.71 mm
- net RP1_CAN_RX: track 0.00 -> 6.95 mm
- net Net-(J1-CC1): track 0.00 -> 6.14 mm
- net Net-(SW7-B): track 0.00 -> 4.64 mm
- net Net-(U2-CE): track 0.00 -> 2.78 mm
- net GND: track 10.8 -> 10.00 mm

Commit message: updates
Parts:
- J3, J4, J5: moved to F.Cu
- moved D14 130.4 mm to (86.0, 76.4), turned to 50 degrees
- moved SW5 121.8 mm to (200.6, 57.4)
- moved SW6 114.5 mm to (203.1, 65.6)
- moved R22 111.8 mm to (88.0, 77.3), turned to -130 degrees
- moved C23 111.2 mm to (88.1, 71.1), turned to 50 degrees
- moved C19 99.8 mm to (127.3, 56.6), turned to 0 degrees
- moved C24 99.5 mm to (93.0, 71.0), turned to 50 degrees
- moved D10 95.5 mm to (121.3, 57.9), turned to 0 degrees
- moved C20 95.2 mm to (130.3, 60.3), turned to 0 degrees
- moved R17 94.9 mm to (120.8, 55.5), turned to 0 degrees
- moved D11 94.7 mm to (157.8, 70.0), turned to 131 degrees
- moved S2 91.6 mm to (135.5, 122.2), turned to -45 degrees
- moved R21 89.1 mm to (83.9, 75.1), turned to 50 degrees
- moved R8 82.5 mm to (148.9, 91.9), turned to 45 degrees
- moved D13 78.7 mm to (89.3, 79.3), turned to -130 degrees
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Routing:
- net +3V3: track 54.0 -> 222.7 mm
- net Net-(J6-Pin_2): track 28.3 -> 117.9 mm
- net Net-(J6-Pin_3): track 30.2 -> 118.7 mm
- net VBUS: track 50.1 -> 79.9 mm
- net ~{RP1_USB_BOOT}: track 0.00 -> 18.5 mm
- net SAO2_TX: track 0.00 -> 9.69 mm
- net SAO1_TX: track 0.00 -> 9.24 mm
- net SAO3_TX: track 0.00 -> 8.45 mm
- net Net-(D2-A): track 0.00 -> 8.11 mm
- net Net-(D10-A): track 0.00 -> 8.08 mm
- net Net-(D11-K): track 0.00 -> 7.83 mm
- net Net-(D13-K): track 0.00 -> 7.32 mm
- net SAO2_RX: track 0.00 -> 6.51 mm
- net SAO1_RX: track 0.00 -> 6.12 mm
- net SAO3_RX: track 0.00 -> 5.30 mm
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
Commit message: closer, but also further
Parts:
- removed SW2, SW3, SW4, SW5, SW6, SW7: SW_SPST, OS102011MS2QN1C:OS102011MS2QN1C
- added S3: MK-12C02-G020, MK-12C02-G020:MK12C02G020, B.Cu at (154.9, 88.2)
- added S4: MK-12C02-G020, MK-12C02-G020:MK12C02G020, B.Cu at (208.8, 83.7)
- added S5: MK-12C02-G020, MK-12C02-G020:MK12C02G020, B.Cu at (208.8, 92.3)
- added S6: MK-12C02-G020, MK-12C02-G020:MK12C02G020, B.Cu at (208.8, 101.0)
- added S7: MK-12C02-G020, MK-12C02-G020:MK12C02G020, B.Cu at (102.6, 115.5)
- added S8: MK-12C02-G020, MK-12C02-G020:MK12C02G020, B.Cu at (110.2, 123.0)
- J4: moved to B.Cu
- moved D13 27.3 mm to (110.2, 97.0), turned to -45 degrees
- moved D9 19.8 mm to (125.6, 81.6), turned to -45 degrees
- moved D11 11.6 mm to (151.9, 80.0), turned to -90 degrees
- moved J1 10.0 mm to (135.7, 133.9)
- moved S2 9.67 mm to (126.7, 126.3), turned to -135 degrees
- moved R3 7.00 mm to (136.9, 122.5), turned to 135 degrees
- moved D1 6.29 mm to (139.3, 125.0), turned to -135 degrees
- moved J6 5.20 mm to (128.3, 135.0), turned to 90 degrees
- moved D3 5.13 mm to (137.6, 86.3), turned to 135 degrees
- moved J4 5.04 mm to (169.7, 64.4), turned to -140 degrees
- moved R23 4.86 mm to (114.0, 118.2), turned to -135 degrees
- moved C10 3.92 mm to (149.8, 121.0)
- moved R4 3.89 mm to (133.3, 123.9), turned to 135 degrees
- moved C2 3.04 mm to (148.1, 125.5)
- moved R9 3.04 mm to (143.2, 126.0)
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Routing:
- net GLOBAL_Silent: track 0.00 -> 67.3 mm
- net Net-(J6-Pin_2): track 117.9 -> 177.5 mm, vias 0 -> 4
- net +3V3: track 222.7 -> 281.1 mm
- net Net-(J6-Pin_3): track 118.7 -> 168.7 mm
- net Net-(D13-K): track 7.32 -> 33.7 mm
- net Net-(D10-A): track 8.08 -> 24.6 mm
- net Net-(D2-A): track 8.11 -> 21.1 mm
- net SAO2_TX: track 9.69 -> 0.00 mm
- net VBUS: track 79.9 -> 70.6 mm
- net Net-(J1-D--PadA7): track 23.1 -> 15.6 mm
- net Net-(J1-D+-PadA6): track 22.3 -> 15.1 mm
- net Net-(D1-A): track 17.4 -> 10.6 mm
- net ~{RP1_USB_BOOT}: track 18.5 -> 21.9 mm
- net Net-(J1-CC2): track 7.71 -> 5.31 mm
- net Net-(R23-Pad2): track 4.64 -> 3.00 mm
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