File: CHV_DC31.kicad_pcb (KiCad board)
At the start: 2 copper layers, 137.3 x 128.4 mm, 102 parts, among them IC1 W25Q16JVUXIQ_TR, J1 USB_C_Receptacle_USB2.0, J2 Conn_01x02, J3 Conn_02x03_Odd_Even, J4 Conn_02x03_Odd_Even, J5 Conn_02x03_Odd_Even, J6 Conn_01x03, Q1 PMOS, U1 MCP2558FD-xMNY, U2 XC6220B331MR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

Commit message: getting closer
Parts:
- moved S1 76.5 mm to (166.8, 124.8), turned to -135 degrees
- moved C20 45.3 mm to (104.2, 38.9)
- moved U4 43.0 mm to (104.7, 35.9), turned to 180 degrees
- moved R18 38.7 mm to (112.8, 33.9)
- moved C19 36.4 mm to (109.6, 37.5), turned to -90 degrees
- moved R22 33.1 mm to (76.6, 66.3), turned to -135 degrees
- moved D10 32.6 mm to (117.5, 34.0), turned to 180 degrees
- moved S4 31.7 mm to (103.9, 45.3), turned to -27 degrees
- moved C24 31.2 mm to (78.7, 60.7)
- moved U6 31.2 mm to (75.3, 62.1)
- moved D14 31.2 mm to (72.6, 64.6)
- moved C23 31.2 mm to (71.3, 60.0)
- moved J5 31.2 mm to (65.9, 57.2)
- moved R21 31.2 mm to (68.5, 62.7)
- moved R17 28.9 mm to (122.0, 33.9)
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- renumbered FIDr to FID1
Connections:
- S4 pad 1: +3V3 -> unconnected-(S4-Pad1)
- S4 pad 3: unconnected-(S4-Pad3) -> +3V3
- S7 pad 2: +3V3 -> unconnected-(S7-Pad2)
- S7 pad 3: unconnected-(S7-Pad3) -> +3V3
Routing:
- net VBUS: track 41.3 -> 128.2 mm
- net Net-(J6-Pin_2): track 154.4 -> 89.4 mm, vias 4 -> 0
- net GLOBAL_Silent: track 34.3 -> 89.7 mm
- net Net-(D10-A): track 32.5 -> 77.6 mm
- net Net-(J6-Pin_3): track 141.5 -> 96.9 mm
- net +3V3: track 438.2 -> 413.9 mm
- net Net-(D11-K): track 17.3 -> 40.6 mm
- net SAO1_RX: track 7.38 -> 26.0 mm
- net Net-(D13-K): track 35.1 -> 53.2 mm
- net SAO1_TX: track 11.0 -> 28.1 mm
- net RUN: track 5.18 -> 11.4 mm

Commit message: almost done!
Parts:
- added R13: R, Resistor_SMD:R_0805_2012Metric, B.Cu at (151.9, 139.2)
- moved C25 113.2 mm to (145.5, 144.5), turned to -45 degrees
- moved U7 112.8 mm to (148.6, 141.3), turned to 45 degrees
- moved Q1 106.1 mm to (145.0, 148.6), turned to 45 degrees
- moved C26 103.5 mm to (153.6, 142.1), turned to 45 degrees
- moved D6 101.8 mm to (148.6, 135.8), turned to 135 degrees
- moved R12 101.2 mm to (142.8, 145.1), turned to 135 degrees
- moved L1 99.3 mm to (143.5, 139.6), turned to 45 degrees
- moved D1 5.10 mm to (140.8, 142.9)
- moved D3 3.57 mm to (148.3, 90.2)
- moved R3 3.51 mm to (139.1, 139.2)
- moved C22 1.25 mm to (182.9, 65.5), turned to -45 degrees
- moved C17 1.18 mm to (158.2, 104.0)
- moved C18 1.18 mm to (162.3, 104.0)
- moved Y1 1.18 mm to (160.2, 105.9)
Connections:
- C26 pad 1: VBUS -> GND
- C26 pad 2: GND -> Net-(C26-Pad2)
- S3 pad 1: Net-(D2-A) -> unconnected-(S3-Pad1)
- S3 pad 2: +3V3 -> Net-(D2-A)
- S3 pad 3: unconnected-(S3-Pad3) -> +3V3
- U7 pad 2: Net-(D6-A) -> VBUS
- U7 pad 3: VBUS -> Net-(D6-A)
Routing:
- net Net-(J6-Pin_2): track 89.4 -> 295.9 mm, vias 0 -> 6
- net Net-(J6-Pin_3): track 96.9 -> 296.7 mm, vias 0 -> 2
- net Net-(BT1-+): track 0.00 -> 162.9 mm, vias 0 -> 2
- net VBUS: track 128.2 -> 244.8 mm, vias 0 -> 2
- net +3V3: track 413.9 -> 438.5 mm, vias 0 -> 2
- net Common_Power: track 13.6 -> 28.6 mm
- net Net-(D6-A): track 0.00 -> 9.19 mm
- net Net-(D1-A): track 13.2 -> 8.93 mm
- net Net-(J1-CC1): track 4.23 -> 7.73 mm
- net USB_POWER: track 0.00 -> 2.94 mm
- net Net-(C26-Pad2): track 0.00 -> 2.34 mm
- net Net-(D2-A): track 21.4 -> 23.1 mm
- net Net-(D11-K): track 40.6 -> 42.1 mm
- net LED_LINE_4: track 50.3 -> 49.3 mm

Commit message: HOLY COW IT'S DONE
Parts:
- moved S6 0.29 mm to (74.9, 79.8)
Connections:
- S7 pad 1: GLOBAL_Silent -> unconnected-(S7-Pad1)
- S7 pad 2: unconnected-(S7-Pad2) -> GLOBAL_Silent
Routing:
- net +3V3: track 438.5 -> 641.6 mm, vias 2 -> 8
- net VBUS: track 244.8 -> 413.6 mm, vias 2 -> 5
- net GND: track 12.4 -> 21.2 mm, vias 0 -> 3
- net Net-(J6-Pin_3): track 296.7 -> 300.1 mm
- net Net-(J6-Pin_2): track 295.9 -> 299.0 mm
- net Net-(D10-A): track 77.6 -> 80.6 mm
- net GLOBAL_Silent: track 89.7 -> 91.6 mm
- net SAO3_TX: track 11.4 -> 10.4 mm
- net Net-(BT1-+): track 162.9 -> 163.4 mm
Other:
- board text added: "Boot Sel"
- board text added: "CANBUS Termination"
- board text added: "GND"
- board text added: "Global Silent"
- board text added: "HIGH"
- board text added: "LOW"
- board text added: "OFF"
- board text added: "ON"
- board text added: "Reset"
