File: CHV_DC31.kicad_sch (KiCad schematic)
At the start: 101 parts, among them IC1 W25Q16JVUXIQ_TR, J1 USB_C_Receptacle_USB2.0, J2 Conn_01x02, J3 Conn_02x03_Odd_Even, J4 Conn_02x03_Odd_Even, J5 Conn_02x03_Odd_Even, J6 Conn_01x03, Q1 PMOS, U1 MCP2558FD-xMNY, U2 XC6220B331MR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

Commit message: HOLY COW IT'S DONE
Connections:
- net GLOBAL_Silent: now also S7.2; no longer S7.1
Changed lines of the file:
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@@
   (no_connect (at 395.224 300.99))
   (no_connect (at 292.862 301.244))
-  (no_connect (at 180.848 330.454))
+  (no_connect (at 180.848 332.994))
   (no_connect (at 143.51 129.286))
   (no_connect (at 143.51 141.986))
@@
     (stroke (width 0) (type default))
   )
-  (wire (pts (xy 180.848 332.994) (xy 184.15 332.994))
+  (wire (pts (xy 180.848 330.454) (xy 184.15 330.454))
     (stroke (width 0) (type default))
   )
@@
     )
   )
-  (global_label "GLOBAL_Silent" (shape input) (at 184.15 332.994 0) (fields_autoplaced)
-    (effects (font (size 1.27 1.27)) (justify left))
-    (property "Intersheetrefs" "${INTERSHEET_REFS}" (at 199.9888 332.9146 0)
+  (global_label "GLOBAL_Silent" (shape input) (at 184.15 330.454 0) (fields_autoplaced)
+    (effects (font (size 1.27 1.27)) (justify left))
+    (property "Intersheetrefs" "${INTERSHEET_REFS}" (at 199.9888 330.3746 0)
       (effects (font (size 1.27 1.27)) (justify left) hide)
     )
@@
     )
     (pin "1")
+    (pin "2")
     (pin "3")
-    (pin "2")
     (instances
       (project "CHV_DC31"

Commit message: We are SOOOOO close
Parts:
- J3, J4, J5: footprint Connector_PinHeader_2.54mm:PinHeader_2x03_P2.54mm_Vertical -> badgelife_sao_v169bis:Badgelife-SAOv169-BADGE-2x3
Changed lines of the file:
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@@
       (effects (font (size 1.27 1.27)))
     )
-    (property "Footprint" "Connector_PinHeader_2.54mm:PinHeader_2x03_P2.54mm_Vertical" (at 361.315 362.585 0)
+    (property "Footprint" "badgelife_sao_v169bis:Badgelife-SAOv169-BADGE-2x3" (at 361.315 362.585 0)
       (effects (font (size 1.27 1.27)) hide)
     )
@@
       (effects (font (size 1.27 1.27)))
     )
-    (property "Footprint" "Connector_PinHeader_2.54mm:PinHeader_2x03_P2.54mm_Vertical" (at 258.064 364.998 0)
+    (property "Footprint" "badgelife_sao_v169bis:Badgelife-SAOv169-BADGE-2x3" (at 258.064 364.998 0)
       (effects (font (size 1.27 1.27)) hide)
     )
@@
       (effects (font (size 1.27 1.27)))
     )
-    (property "Footprint" "Connector_PinHeader_2.54mm:PinHeader_2x03_P2.54mm_Vertical" (at 458.724 360.68 0)
-      (effects (font (size 1.27 1.27)) hide)
-    )
+    (property "Footprint" "badgelife_sao_v169bis:Badgelife-SAOv169-BADGE-2x3" (at 458.724 360.68 0)
+      (effects (font (size 1.27 1.27)) hide)
+    )

Commit message: added countersink leds
Parts:
- D15, D16, D17, D18, D19, D20, D21, D22, D23: footprint LED_SMD:LED_1206_3216Metric -> engine:P2-1206RTCS2-0.9T-F
Changed lines of the file:
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@@
       (effects (font (size 1.27 1.27)))
     )
-    (property "Footprint" "LED_SMD:LED_1206_3216Metric" (at 339.598 62.738 0)
+    (property "Footprint" "engine:P2-1206RTCS2-0.9T-F" (at 339.598 62.738 0)
       (effects (font (size 1.27 1.27)) hide)
     )
@@
       (effects (font (size 1.27 1.27)))
     )
-    (property "Footprint" "LED_SMD:LED_1206_3216Metric" (at 307.34 62.738 0)
+    (property "Footprint" "engine:P2-1206RTCS2-0.9T-F" (at 307.34 62.738 0)
       (effects (font (size 1.27 1.27)) hide)
     )
@@
       (effects (font (size 1.27 1.27)))
     )
-    (property "Footprint" "LED_SMD:LED_1206_3216Metric" (at 290.83 62.738 0)
+    (property "Footprint" "engine:P2-1206RTCS2-0.9T-F" (at 290.83 62.738 0)
       (effects (font (size 1.27 1.27)) hide)
     )
@@
       (effects (font (size 1.27 1.27)))
     )
-    (property "Footprint" "LED_SMD:LED_1206_3216Metric" (at 347.472 62.738 0)
+    (property "Footprint" "engine:P2-1206RTCS2-0.9T-F" (at 347.472 62.738 0)
       (effects (font (size 1.27 1.27)) hide)
     )
@@
       (effects (font (size 1.27 1.27)))
     )
-    (property "Footprint" "LED_SMD:LED_1206_3216Metric" (at 315.214 62.738 0)
+    (property "Footprint" "engine:P2-1206RTCS2-0.9T-F" (at 315.214 62.738 0)
       (effects (font (size 1.27 1.27)) hide)
     )
@@
       (effects (font (size 1.27 1.27)))
     )
-    (property "Footprint" "LED_SMD:LED_1206_3216Metric" (at 331.47 62.738 0)
+    (property "Footprint" "engine:P2-1206RTCS2-0.9T-F" (at 331.47 62.738 0)
       (effects (font (size 1.27 1.27)) hide)
     )
@@
       (effects (font (size 1.27 1.27)))
     )
-    (property "Footprint" "LED_SMD:LED_1206_3216Metric" (at 282.702 62.738 0)
+    (property "Footprint" "engine:P2-1206RTCS2-0.9T-F" (at 282.702 62.738 0)
       (effects (font (size 1.27 1.27)) hide)
     )
@@
       (effects (font (size 1.27 1.27)))
     )
-    (property "Footprint" "LED_SMD:LED_1206_3216Metric" (at 323.088 62.738 0)
+    (property "Footprint" "engine:P2-1206RTCS2-0.9T-F" (at 323.088 62.738 0)
       (effects (font (size 1.27 1.27)) hide)
     )
@@
       (effects (font (size 1.27 1.27)))
     )
-    (property "Footprint" "LED_SMD:LED_1206_3216Metric" (at 298.958 62.738 0)
-      (effects (font (size 1.27 1.27)) hide)
-    )
+    (property "Footprint" "engine:P2-1206RTCS2-0.9T-F" (at 298.958 62.738 0)
+      (effects (font (size 1.27 1.27)) hide)
+    )

Commit message: finished
Other:
- note added: "New"
- moved on the sheet: BT1, C25, C26, D6, L1, Q1, R12, R13, U7

Commit message: Holy cow, done
Parts:
- removed R13: R, Resistor_SMD:R_0805_2012Metric, symbol Device:R
- L1: footprint Inductor_SMD:L_0805_2012Metric -> engine:inductor_tmp
- U7: footprint Package_TO_SOT_SMD:SOT-89-3 -> Package_TO_SOT_SMD:SOT-23
Connections:
- net Common_Power: no longer C2.1, R9.1, U2.1 (VIN)
- net USB_POWER: now also D1.2 (A), J1.A4 (VBUS), J1.A9 (VBUS), J1.B4 (VBUS), J1.B9 (VBUS)
- net VBUS: now also C2.1, C26.2, R9.1, U2.1 (VIN)
Other:
- moved on the sheet: C10, C2, R9, U2
